File: pcb/suntastic/mppt_charger.kicad_sch (KiCad schematic)
At the start: 0 parts

Commit message: Add screw terminals for external MPPT module and PV input
Parts:
- added J3: INPUT FROM EXT MPPT, TerminalBlock:TerminalBlock_bornier-2_P5.08mm, symbol Connector:Screw_Terminal_01x02
- added J3: OUT TO EXT MPPT, TerminalBlock:TerminalBlock_bornier-2_P5.08mm, symbol Connector:Screw_Terminal_01x02
- added JP18 (x2): Jumper_2_Open, Jumper:SolderJumper-2_P1.3mm_Open_RoundedPad1.0x1.5mm, symbol Jumper:Jumper_2_Open
- added TP15: OUT_FROM_MPPT, TestPoint:TestPoint_THTPad_4.0x4.0mm_Drill2.0mm, symbol Connector:TestPoint
- added TP15: GND_TO_MPPT, TestPoint:TestPoint_THTPad_4.0x4.0mm_Drill2.0mm, symbol Connector:TestPoint
- added TP15: GND_FROM_MPPT, TestPoint:TestPoint_THTPad_4.0x4.0mm_Drill2.0mm, symbol Connector:TestPoint
- added TP15: PV_TO_MPPT, TestPoint:TestPoint_THTPad_4.0x4.0mm_Drill2.0mm, symbol Connector:TestPoint
Connections:
- new net: J3.1 (Pin_1), JP18.1 (A), TP15.1
- new net: J3.2 (Pin_2), JP18.1 (A), TP15.1
- new net GND: JP18.2 (B), JP18.2 (B)
- new net MPPT_OUT: J3.2 (Pin_2), TP15.1
- new net PV_+: J3.1 (Pin_1), TP15.1
