File: pcb/suntastic/solar_panel_input.kicad_sch (KiCad schematic)
At the start: 0 parts

Commit message: Add screw terminals for external MPPT module and PV input
Parts:
- added J3: PV IN, TerminalBlock:TerminalBlock_bornier-2_P5.08mm, symbol Connector:Screw_Terminal_01x02
- added JP18: Jumper_2_Open, Jumper:SolderJumper-2_P1.3mm_Open_RoundedPad1.0x1.5mm, symbol Jumper:Jumper_2_Open
- added TP15: PV_VIN, TestPoint:TestPoint_THTPad_4.0x4.0mm_Drill2.0mm, symbol Connector:TestPoint
- added TP15: PV_GND, TestPoint:TestPoint_THTPad_4.0x4.0mm_Drill2.0mm, symbol Connector:TestPoint
Connections:
- new net: J3.1 (Pin_1), JP18.1 (A), TP15.1
- new net GND: JP18.2 (B)
- new net PV_+: J3.2 (Pin_2), TP15.1
Changed lines of the file:
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@@
     (rev "1")
   )
+  (junction (at 129.4384 76.454) (diameter 0) (color 0 0 0 0)
+  )
+  (junction (at 123.063 70.104) (diameter 0) (color 0 0 0 0)
+  )
+  (wire (pts (xy 125.73 76.454) (xy 129.4384 76.454))
+    (stroke (width 0) (type default))
+  )
+  (wire (pts (xy 129.4384 75.438) (xy 129.4384 76.454))
+    (stroke (width 0) (type default))
+  )
+  (wire (pts (xy 123.19 70.104) (xy 123.19 77.089))
+    (stroke (width 0) (type default))
+  )
+  (wire (pts (xy 123.063 70.104) (xy 123.19 70.104))
+    (stroke (width 0) (type default))
+  )
+  (wire (pts (xy 118.745 70.104) (xy 123.063 70.104))
+    (stroke (width 0) (type default))
+  )
+  (wire (pts (xy 125.73 76.454) (xy 125.73 77.089))
+    (stroke (width 0) (type default))
+  )
+  (wire (pts (xy 129.4384 64.262) (xy 129.413 64.262))
+    (stroke (width 0) (type default))
+  )
+  (wire (pts (xy 129.4384 76.454) (xy 129.54 76.454))
+    (stroke (width 0) (type default))
+  )
+  (wire (pts (xy 129.4384 65.278) (xy 129.4384 64.262))
+    (stroke (width 0) (type default))
+  )
+  (wire (pts (xy 123.063 68.707) (xy 123.063 70.104))
+    (stroke (width 0) (type default))
+  )
+  (global_label "PV_+" (shape input) (at 123.063 68.707 90) (fields_autoplaced)
+    (effects (font (size 1.27 1.27)) (justify left))
+    (property "Intersheetrefs" "${INTERSHEET_REFS}" (at 123.063 60.9026 90)
+      (effects (font (size 1.27 1.27)) (justify left) hide)
+    )
+  )
+  (symbol (lib_id "Connector:Screw_Terminal_01x02") (at 125.73 82.169 270) (unit 1)
+    (in_bom yes) (on_board yes) (dnp no)
+    (property "Reference" "J3" (at 122.809 84.963 90)
+      (effects (font (size 1.27 1.27)) (justify left))
+    )
+    (property "Value" "PV IN" (at 122.047 86.741 90)
+      (effects (font (size 1.27 1.27)) (justify left))
+    )
+    (property "Footprint" "TerminalBlock:TerminalBlock_bornier-2_P5.08mm" (at 125.73 82.169 0)
+      (effects (font (size 1.27 1.27)) hide)
+    )
+    (property "Datasheet" "~" (at 125.73 82.169 0)
+      (effects (font (size 1.27 1.27)) hide)
+    )
+    (pin "1")
+    (pin "2")
+    (instances
+      (project "suntastic"
+        (path "/4d5a6178-89d6-4824-ac30-5dee40aabff2/70576ca8-d50a-4f6d-b4d0-36474c2d5281"
+          (reference "J3") (unit 1)
+        )
+        (path "/4d5a6178-89d6-4824-ac30-5dee40aabff2/d7e9a640-ff81-456c-bdbb-c4d60fbd13c6"
+          (reference "J12") (unit 1)
+        )
+      )
+    )
+  )
+  (symbol (lib_id "Jumper:Jumper_2_Open") (at 129.4384 70.358 90) (unit 1)
+    (in_bom yes) (on_board yes) (dnp no)
+    (property "Reference" "JP18" (at 130.9624 69.342 90)
+      (effects (font (size 1.27 1.27)) (justify right))
+    )
+    (property "Value" "Jumper_2_Open" (at 130.7084 71.628 90)
+      (effects (font (size 1.27 1.27)) (justify right))
+    )
+    (property "Footprint" "Jumper:SolderJumper-2_P1.3mm_Open_RoundedPad1.0x1.5mm" (at 129.4384 70.358 0)
+      (effects (font (size 1.27 1.27)) hide)
+    )
+    (property "Datasheet" "~" (at 129.4384 70.358 0)
+      (effects (font (size 1.27 1.27)) hide)
+    )
+    (pin "1")
+    (pin "2")
+    (instances
+      (project "suntastic"
+        (path "/4d5a6178-89d6-4824-ac30-5dee40aabff2/70576ca8-d50a-4f6d-b4d0-36474c2d5281"
+          (reference "JP18") (unit 1)
+        )
+        (path "/4d5a6178-89d6-4824-ac30-5dee40aabff2/0be65f9d-b3fc-407f-86f4-ba5a551916f5"
+          (reference "JP29") (unit 1)
+        )
+        (path "/4d5a6178-89d6-4824-ac30-5dee40aabff2/d7e9a640-ff81-456c-bdbb-c4d60fbd13c6"
+          (reference "JP31") (unit 1)
+        )
+      )
+    )
+  )
+  (symbol (lib_id "Connector:TestPoint") (at 118.745 70.104 90) (unit 1)
+    (in_bom yes) (on_board yes) (dnp no)
+    (property "Reference" "TP15" (at 115.57 77.724 0)
+      (effects (font (size 1.27 1.27)) (justify left))
+    )
+    (property "Value" "PV_VIN" (at 118.11 77.724 0)
+      (effects (font (size 1.27 1.27)) (justify left))
+    )
+    (property "Footprint" "TestPoint:TestPoint_THTPad_4.0x4.0mm_Drill2.0mm" (at 118.745 65.024 0)
+      (effects (font (size 1.27 1.27)) hide)
+    )
+    (property "Datasheet" "~" (at 118.745 65.024 0)
+      (effects (font (size 1.27 1.27)) hide)
+    )
+    (pin "1")
+    (instances
+      (project "suntastic"
+        (path "/4d5a6178-89d6-4824-ac30-5dee40aabff2/fadcfaa3-5ba9-44dc-a564-21a258e74f25"
+          (reference "TP15") (unit 1)
+        )
+        (path "/4d5a6178-89d6-4824-ac30-5dee40aabff2/70576ca8-d50a-4f6d-b4d0-36474c2d5281"
+          (reference "TP19") (unit 1)
+        )
+        (path "/4d5a6178-89d6-4824-ac30-5dee40aabff2/d7e9a640-ff81-456c-bdbb-c4d60fbd13c6"
+          (reference "TP10") (unit 1)
+        )
+      )
+    )
+  )
+  (symbol (lib_id "Connector:TestPoint") (at 129.54 76.454 270) (unit 1)
+    (in_bom yes) (on_board yes) (dnp no)
+    (property "Reference" "TP15" (at 132.715 78.994 0)
+      (effects (font (size 1.27 1.27)) (justify left))
+    )
+    (property "Value" "PV_GND" (at 130.81 78.994 0)
+      (effects (font (size 1.27 1.27)) (justify left))
+    )
+    (property "Footprint" "TestPoint:TestPoint_THTPad_4.0x4.0mm_Drill2.0mm" (at 129.54 81.534 0)
+      (effects (font (size 1.27 1.27)) hide)
+    )
+    (property "Datasheet" "~" (at 129.54 81.534 0)
+      (effects (font (size 1.27 1.27)) hide)
+    )
+    (pin "1")
+    (instances
+      (project "suntastic"
+        (path "/4d5a6178-89d6-4824-ac30-5dee40aabff2/fadcfaa3-5ba9-44dc-a564-21a258e74f25"
+          (reference "TP15") (unit 1)
+        )
+        (path "/4d5a6178-89d6-4824-ac30-5dee40aabff2/70576ca8-d50a-4f6d-b4d0-36474c2d5281"
+          (reference "TP20") (unit 1)
+        )
+        (path "/4d5a6178-89d6-4824-ac30-5dee40aabff2/d7e9a640-ff81-456c-bdbb-c4d60fbd13c6"
+          (reference "TP11") (unit 1)
+        )
+      )
+    )
+  )
+  (symbol (lib_id "power:GND") (at 129.413 64.262 180) (unit 1)
+    (in_bom yes) (on_board yes) (dnp no) (fields_autoplaced)
+    (property "Reference" "#PWR026" (at 129.413 57.912 0)
+      (effects (font (size 1.27 1.27)) hide)
+    )
+    (property "Value" "GND" (at 129.413 60.452 0)
+      (effects (font (size 1.27 1.27)))
+    )
+    (property "Footprint" "" (at 129.413 64.262 0)
+      (effects (font (size 1.27 1.27)) hide)
+    )
+    (property "Datasheet" "" (at 129.413 64.262 0)
+      (effects (font (size 1.27 1.27)) hide)
+    )
+    (pin "1")
+    (instances
+      (project "suntastic"
+        (path "/4d5a6178-89d6-4824-ac30-5dee40aabff2/70576ca8-d50a-4f6d-b4d0-36474c2d5281"
+          (reference "#PWR026") (unit 1)
+        )
+        (path "/4d5a6178-89d6-4824-ac30-5dee40aabff2/d7e9a640-ff81-456c-bdbb-c4d60fbd13c6"
+          (reference "#PWR056") (unit 1)
+        )
+      )
+    )
+  )
 )
